Commit message: implemented plane mobility scheme and trajectory saving algorithms

File: myur5sim/myur5_description/urdf/person.urdf.xacro (robot description, xacro)
@@ -44,5 +44,5 @@
     <parent link="world" />
     <child link = "chair_base" />
-    <origin xyz="0.0 0.78 0.15" rpy="0.0 0.0 0.0" />
+    <origin xyz="0.78 0.78 0.15" rpy="0.0 0.0 0.785" />
   </joint>
 <!--

File: myur5sim/myur5_description/urdf/scalable_person.urdf.xacro (robot description, xacro)
@@ -47,5 +47,5 @@
     <parent link="world" />
     <child link = "chair_base" />
-    <origin xyz="0.0 0.78 0.15" rpy="0.0 0.0 0.0" />
+    <origin xyz="0.78 0.78 0.15" rpy="0.0 0.0 -0.785" />
   </joint>
 <!-- Hip -->
